File: KICAD/droidrone.kicad_pcb (KiCad board)
At the start: 2 copper layers, 100 x 50 mm, 68 parts, among them IC1 ATMEGA328PB, P1 USB_A, U1 TA4805S, U2 ITEAD_HC-05, U4 LP2950L-3.3V, Y1 Crystal

Commit message: 配線開始
Parts:
- removed 0.1uF4: 0.1uF, Capacitors_ThroughHole:C_Rect_L4.0mm_W2.5mm_P2.50mm
- removed 100uF10V1: 100uF 10V, Capacitors_ThroughHole:CP_Radial_D8.0mm_P2.50mm
- removed 10k4: 10k, Resistors_ThroughHole:R_Axial_DIN0204_L3.6mm_D1.6mm_P2.54mm_Vertical
- removed 1k6: 1k, Resistors_ThroughHole:R_Axial_DIN0204_L3.6mm_D1.6mm_P2.54mm_Vertical
- removed D17: CONN_01X03, Pin_Headers:Pin_Header_Straight_1x03_Pitch2.54mm
- removed HC05S1: LED, LEDs:LED_D5.0mm
- removed No-BEC1: JUMPER, Pin_Headers:Pin_Header_Straight_1x02_Pitch2.54mm
- removed U1: TA4805S, TO_SOT_Packages_THT:TO-220_Neutral123_Vertical_LargePads
- added ?: MountingHole_3.2mm_M3, Mounting_Holes:MountingHole_3.2mm_M3, F.Cu at (190.0, 70.0)
- added ?: Hole_1.0mm, lib:Hole_1.0mm, F.Cu at (194.0, 32.5)
- added ?: Hole_1.0mm, lib:Hole_1.0mm, F.Cu at (194.0, 44.5)
- added ?: Hole_1.0mm, lib:Hole_1.0mm, F.Cu at (194.0, 46.0)
- added ?: Hole_1.0mm, lib:Hole_1.0mm, F.Cu at (194.0, 47.5)
- added ?: Hole_1.0mm, lib:Hole_1.0mm, F.Cu at (194.0, 43.0)
- added ?: Hole_1.0mm, lib:Hole_1.0mm, F.Cu at (194.0, 37.0)
- added ?: Hole_1.0mm, lib:Hole_1.0mm, F.Cu at (194.0, 41.5)
- added ?: Hole_1.0mm, lib:Hole_1.0mm, F.Cu at (194.0, 40.0)
- added ?: Hole_1.0mm, lib:Hole_1.0mm, F.Cu at (194.0, 38.5)
- added ?: Hole_1.0mm, lib:Hole_1.0mm, F.Cu at (194.0, 49.0)
- added ?: MountingHole_3.2mm_M3, Mounting_Holes:MountingHole_3.2mm_M3, F.Cu at (190.0, 30.0)
- added ?: Hole_1.0mm, lib:Hole_1.0mm, F.Cu at (194.0, 74.5)
- added ?: Hole_1.0mm, lib:Hole_1.0mm, F.Cu at (194.0, 64.0)
- added ?: Hole_1.0mm, lib:Hole_1.0mm, F.Cu at (194.0, 65.5)
- added ?: Hole_1.0mm, lib:Hole_1.0mm, F.Cu at (194.0, 67.0)
- added ?: Hole_1.0mm, lib:Hole_1.0mm, F.Cu at (194.0, 62.5)
- added ?: Hole_1.0mm, lib:Hole_1.0mm, F.Cu at (194.0, 68.5)
- added ?: Hole_1.0mm, lib:Hole_1.0mm, F.Cu at (194.0, 73.0)
- added ?: Hole_1.0mm, lib:Hole_1.0mm, F.Cu at (194.0, 71.5)
- added ?: Hole_1.0mm, lib:Hole_1.0mm, F.Cu at (194.0, 70.0)
- added ?: Hole_1.0mm, lib:Hole_1.0mm, F.Cu at (194.0, 58.0)
- added ?: MountingHole_3.2mm_M3, Mounting_Holes:MountingHole_3.2mm_M3, F.Cu at (130.0, 30.0)
- added ?: Hole_1.0mm, lib:Hole_1.0mm, F.Cu at (194.0, 59.5)
- added ?: Hole_1.0mm, lib:Hole_1.0mm, F.Cu at (194.0, 61.0)
- added ?: Hole_1.0mm, lib:Hole_1.0mm, F.Cu at (194.0, 56.5)
- added ?: Hole_1.0mm, lib:Hole_1.0mm, F.Cu at (197.0, 50.5)
- added ?: Hole_1.0mm, lib:Hole_1.0mm, F.Cu at (195.5, 50.5)
- added ?: Hole_1.0mm, lib:Hole_1.0mm, F.Cu at (194.0, 50.5)
- added ?: Hole_1.0mm, lib:Hole_1.0mm, F.Cu at (194.0, 55.0)
- added ?: Hole_1.0mm, lib:Hole_1.0mm, F.Cu at (194.0, 53.5)
- added ?: Hole_1.0mm, lib:Hole_1.0mm, F.Cu at (194.0, 52.0)
- added ?: Hole_1.0mm, lib:Hole_1.0mm, F.Cu at (201.5, 50.5)
- added ?: Hole_1.0mm, lib:Hole_1.0mm, F.Cu at (194.0, 26.5)
- added ?: Hole_1.0mm, lib:Hole_1.0mm, F.Cu at (200.0, 50.5)
- added ?: Hole_1.0mm, lib:Hole_1.0mm, F.Cu at (198.5, 50.5)
- added ?: Hole_1.0mm, lib:Hole_1.0mm, F.Cu at (203.0, 50.5)
- added ?: Hole_1.0mm, lib:Hole_1.0mm, F.Cu at (204.5, 50.5)
- added ?: Hole_1.0mm, lib:Hole_1.0mm, F.Cu at (206.0, 50.5)
- added ?: Hole_1.0mm, lib:Hole_1.0mm, F.Cu at (224.0, 50.5)
- added ?: Hole_1.0mm, lib:Hole_1.0mm, F.Cu at (222.5, 50.5)
- added ?: Hole_1.0mm, lib:Hole_1.0mm, F.Cu at (221.0, 50.5)
- added ?: Hole_1.0mm, lib:Hole_1.0mm, F.Cu at (216.5, 50.5)
- added ?: Hole_1.0mm, lib:Hole_1.0mm, F.Cu at (218.0, 50.5)
- added ?: Hole_1.0mm, lib:Hole_1.0mm, F.Cu at (194.0, 28.0)
- added ?: Hole_1.0mm, lib:Hole_1.0mm, F.Cu at (219.5, 50.5)
- added ?: Hole_1.0mm, lib:Hole_1.0mm, F.Cu at (210.5, 50.5)
- added ?: Hole_1.0mm, lib:Hole_1.0mm, F.Cu at (209.0, 50.5)
- added ?: Hole_1.0mm, lib:Hole_1.0mm, F.Cu at (207.5, 50.5)
- added ?: Hole_1.0mm, lib:Hole_1.0mm, F.Cu at (212.0, 50.5)
- added ?: Hole_1.0mm, lib:Hole_1.0mm, F.Cu at (213.5, 50.5)
- added ?: Hole_1.0mm, lib:Hole_1.0mm, F.Cu at (215.0, 50.5)
- added ?: MountingHole_3.2mm_M3, Mounting_Holes:MountingHole_3.2mm_M3, F.Cu at (130.0, 70.0)
- added ?: Hole_1.0mm, lib:Hole_1.0mm, F.Cu at (194.0, 29.5)
- added ?: Hole_1.0mm, lib:Hole_1.0mm, F.Cu at (194.0, 31.0)
- added ?: Hole_1.0mm, lib:Hole_1.0mm, F.Cu at (194.0, 35.5)
- added ?: Hole_1.0mm, lib:Hole_1.0mm, F.Cu at (194.0, 34.0)
- 6V-IN1: footprint lib:TB-2pin -> Pin_Headers:Pin_Header_Straight_1x02_Pitch2.54mm
- RX TX GND 5V: renamed from SPP5V1
- Y1: footprint Crystals:Crystal_HC49-U-3pin_Vertical -> lib:Crystal_HC49-U-3pin_Vertical
- moved 1k5 76.9 mm to (181.0, 70.0), turned to 180 degrees
- moved 1k4 76.7 mm to (181.0, 64.0), turned to 180 degrees
- moved 0.1uF1 75.0 mm to (177.0, 31.0)
- moved GroveAna1 73.3 mm to (171.0, 28.0), turned to 90 degrees
- moved 10k3 66.6 mm to (155.0, 26.0)
- moved 2.2k4 63.3 mm to (145.0, 35.0), turned to 180 degrees
- moved 2.2k5 61.2 mm to (145.0, 37.0), turned to 180 degrees
- moved 10k1 56.2 mm to (155.0, 29.0)
- moved 47uF10V1 55.3 mm to (186.0, 34.0), turned to 180 degrees
- moved 2.2k3 53.4 mm to (145.0, 39.0), turned to 180 degrees
- moved Reset1 52.0 mm to (138.0, 29.0)
- moved 2.2k2 49.6 mm to (145.0, 41.0), turned to 180 degrees
- moved 10k5 45.5 mm to (208.2, 54.0), turned to 180 degrees
- moved UART1 44.4 mm to (154.0, 37.0), turned to 90 degrees
- moved 1k8 41.0 mm to (167.0, 41.0), turned to 180 degrees
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Connections:
- net +6V renamed Net-(10k3-Pad1)
- 2.2k3 pad 1: Net-(2.2k3-Pad1) -> +5V
- 2.2k3 pad 2: +5V -> Net-(2.2k3-Pad2)
- 22pF2 pad 1: GND -> Net-(22pF2-Pad1)
- 22pF2 pad 2: Net-(22pF2-Pad2) -> GND
- D10 pad 2: +5VA -> +5V
- D12 pad 2: +5VA -> +5V
- D13 pad 2: +5VA -> +5V
- D2 pad 2: +5VA -> +5V
- D4 pad 2: +5VA -> +5V
- D7 pad 2: +5VA -> +5V
- D8 pad 2: +5VA -> +5V
- D9 pad 2: +5VA -> +5V
- GrI2C-S1 pad 3: Net-(2.2k3-Pad1) -> Net-(2.2k3-Pad2)
- IC1 pad 3: Net-(2.2k3-Pad1) -> Net-(2.2k3-Pad2)
- IC1 pad 8: Net-(22pF2-Pad2) -> Net-(22pF2-Pad1)
- P1 pad 2: (no net) -> Net-(P1-Pad2)
- P1 pad 3: (no net) -> Net-(P1-Pad3)
- RN4020 pad 11: (no net) -> Net-(RN4020-Pad11)
- RN4020 pad 13: (no net) -> Net-(RN4020-Pad13)
- RN4020 pad 14: (no net) -> Net-(RN4020-Pad14)
- RN4020 pad 17: (no net) -> Net-(RN4020-Pad17)
- RN4020 pad 18: (no net) -> Net-(RN4020-Pad18)
- RN4020 pad 19: (no net) -> Net-(RN4020-Pad19)
- RN4020 pad 2: (no net) -> Net-(RN4020-Pad2)
- RN4020 pad 20: (no net) -> Net-(RN4020-Pad20)
- RN4020 pad 21: (no net) -> Net-(RN4020-Pad21)
- RN4020 pad 22: (no net) -> Net-(RN4020-Pad22)
- RN4020 pad 3: (no net) -> Net-(RN4020-Pad3)
- RN4020 pad 4: (no net) -> Net-(RN4020-Pad4)
- RN42XV1 pad 11: (no net) -> Net-(RN42XV1-Pad11)
- RN42XV1 pad 13: (no net) -> Net-(RN42XV1-Pad13)
- RN42XV1 pad 14: (no net) -> Net-(RN42XV1-Pad14)
- RN42XV1 pad 15: (no net) -> Net-(RN42XV1-Pad15)
- RN42XV1 pad 17: (no net) -> Net-(RN42XV1-Pad17)
- RN42XV1 pad 18: (no net) -> Net-(RN42XV1-Pad18)
- RN42XV1 pad 19: (no net) -> Net-(RN42XV1-Pad19)
- RN42XV1 pad 20: (no net) -> Net-(RN42XV1-Pad20)
- RN42XV1 pad 4: (no net) -> Net-(RN42XV1-Pad4)
- RN42XV1 pad 5: (no net) -> Net-(RN42XV1-Pad5)
- RN42XV1 pad 6: (no net) -> Net-(RN42XV1-Pad6)
- RN42XV1 pad 7: (no net) -> Net-(RN42XV1-Pad7)
- RN42XV1 pad 8: (no net) -> Net-(RN42XV1-Pad8)
- RN42XV1 pad 9: (no net) -> Net-(RN42XV1-Pad9)
- RN42XV2 pad 11: (no net) -> Net-(RN42XV2-Pad11)
- RN42XV2 pad 12: (no net) -> Net-(RN42XV2-Pad12)
- RN42XV2 pad 13: (no net) -> Net-(RN42XV2-Pad13)
- RN42XV2 pad 14: (no net) -> Net-(RN42XV2-Pad14)
- RN42XV2 pad 15: (no net) -> Net-(RN42XV2-Pad15)
- RN42XV2 pad 16: (no net) -> Net-(RN42XV2-Pad16)
- RN42XV2 pad 17: (no net) -> Net-(RN42XV2-Pad17)
- RN42XV2 pad 18: (no net) -> Net-(RN42XV2-Pad18)
- RN42XV2 pad 19: (no net) -> Net-(RN42XV2-Pad19)
- RN42XV2 pad 20: (no net) -> Net-(RN42XV2-Pad20)
- RN42XV2 pad 4: (no net) -> Net-(RN42XV2-Pad4)
- RN42XV2 pad 5: (no net) -> Net-(RN42XV2-Pad5)
- RN42XV2 pad 6: (no net) -> Net-(RN42XV2-Pad6)
- RN42XV2 pad 7: (no net) -> Net-(RN42XV2-Pad7)
- RN42XV2 pad 8: (no net) -> Net-(RN42XV2-Pad8)
- RN42XV2 pad 9: (no net) -> Net-(RN42XV2-Pad9)
- U2 pad 10: (no net) -> Net-(U2-Pad10)
- U2 pad 15: (no net) -> Net-(U2-Pad15)
- U2 pad 16: (no net) -> Net-(U2-Pad16)
- U2 pad 17: (no net) -> Net-(U2-Pad17)
- U2 pad 18: (no net) -> Net-(U2-Pad18)
- U2 pad 19: (no net) -> Net-(U2-Pad19)
- U2 pad 20: (no net) -> Net-(U2-Pad20)
- U2 pad 23: (no net) -> Net-(U2-Pad23)
- U2 pad 25: (no net) -> Net-(U2-Pad25)
- U2 pad 27: (no net) -> Net-(U2-Pad27)
- U2 pad 28: (no net) -> Net-(U2-Pad28)
- U2 pad 29: (no net) -> Net-(U2-Pad29)
- U2 pad 3: (no net) -> Net-(U2-Pad3)
- U2 pad 30: (no net) -> Net-(U2-Pad30)
- U2 pad 33: (no net) -> Net-(U2-Pad33)
- U2 pad 4: (no net) -> Net-(U2-Pad4)
- U2 pad 5: (no net) -> Net-(U2-Pad5)
- U2 pad 6: (no net) -> Net-(U2-Pad6)
- U2 pad 7: (no net) -> Net-(U2-Pad7)
- U2 pad 8: (no net) -> Net-(U2-Pad8)
- U2 pad 9: (no net) -> Net-(U2-Pad9)
- Y1 pad 1: Net-(22pF2-Pad2) -> Net-(22pF2-Pad1)
- Y1 pad 3: (no net) -> GND
Routing:
- net +5V: track 0.00 -> 68.0 mm
- net Net-(Conn1-Pad1): track 0.00 -> 66.7 mm
- net GND: track 0.00 -> 63.6 mm
- net Net-(1k7-Pad2): track 0.00 -> 38.5 mm
- net /D2: track 0.00 -> 36.1 mm
- net /D4: track 0.00 -> 35.7 mm
- net Net-(10k5-Pad2): track 0.00 -> 34.6 mm
- net Net-(SPP5V1-Pad2): track 0.00 -> 31.7 mm
- net Net-(RN4020-Pad15): track 0.00 -> 30.6 mm, vias 0 -> 2
- net Net-(SPP5V1-Pad1): track 0.00 -> 30.5 mm
- net /D16/A2: track 0.00 -> 29.6 mm, vias 0 -> 1
- net /D13: track 0.00 -> 27.3 mm, vias 0 -> 1
- net Net-(State1-Pad2): track 0.00 -> 27.3 mm
- net /D7: track 0.00 -> 25.9 mm
- net /D12: track 0.00 -> 25.9 mm
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Other:
- net class 5VA added: clearance 0.2, trace_width 1, via_dia 1.2, via_drill 0.6

Commit message: 配線終了
Parts:
- moved GroveAna1 11.1 mm to (160.6, 31.8)
- moved 1k8 9.60 mm to (157.4, 41.0)
- moved 2.2k2 7.53 mm to (142.8, 48.2), turned to 0 degrees
- moved GrI2C-S1 7.42 mm to (140.8, 42.2), turned to 90 degrees
- moved 2.2k3 7.15 mm to (142.8, 45.8), turned to 0 degrees
- moved 10k3 6.21 mm to (149.8, 29.4)
- moved 10k2 6.05 mm to (143.0, 34.8), turned to 180 degrees
- moved 10k1 5.65 mm to (149.8, 26.8)
- moved 2.2k4 5.46 mm to (142.8, 40.0), turned to 90 degrees
- moved 2.2k5 5.33 mm to (140.6, 40.0), turned to 90 degrees
- moved 1k3 5.00 mm to (171.0, 36.0)
- moved 0.1uF6 4.06 mm to (151.4, 44.4), turned to 90 degrees
- moved 0.1uF5 3.05 mm to (152.4, 34.6), turned to 0 degrees
- moved 2.2k1 3.00 mm to (171.0, 33.0)
- moved 3.3k1 3.00 mm to (171.0, 30.0)
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Connections:
- P1 pad 5: Net-(P1-Pad5) -> (no net)
Routing:
- net GND: track 63.6 -> 323.1 mm
- net +5V: track 68.0 -> 256.2 mm, vias 0 -> 2
- net Net-(0.1uF5-Pad2): track 0.00 -> 57.9 mm, vias 0 -> 1
- net /D18/A4/SDA: track 0.00 -> 39.4 mm
- net /D19/A5/SCL: track 0.00 -> 38.2 mm
- net Net-(1k8-Pad1): track 0.00 -> 38.1 mm
- net Net-(1k3-Pad2): track 0.00 -> 33.1 mm
- net /D11(P): track 0.00 -> 30.4 mm, vias 0 -> 1
- net /TXD: track 0.00 -> 27.9 mm, vias 0 -> 1
- net /D17/A3: track 0.00 -> 25.0 mm
- net /RXD: track 0.00 -> 23.7 mm, vias 0 -> 1
- net Net-(2.2k2-Pad2): track 0.00 -> 18.3 mm, vias 0 -> 1
- net Net-(2.2k1-Pad2): track 0.00 -> 17.5 mm
- net /D13: track 27.3 -> 43.6 mm
- net Net-(2.2k3-Pad2): track 0.00 -> 15.5 mm, vias 0 -> 1
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
Commit message: 配線終了2
Parts:
- removed the ? at (194.0, 32.5)
- removed the ? at (194.0, 44.5)
- removed the ? at (194.0, 46.0)
- removed the ? at (194.0, 47.5)
- removed the ? at (194.0, 43.0)
- removed the ? at (194.0, 37.0)
- removed the ? at (194.0, 41.5)
- removed the ? at (194.0, 40.0)
- removed the ? at (194.0, 38.5)
- removed the ? at (194.0, 49.0)
- removed the ? at (194.0, 74.5)
- removed the ? at (194.0, 64.0)
- removed the ? at (194.0, 65.5)
- removed the ? at (194.0, 67.0)
- removed the ? at (194.0, 62.5)
- removed the ? at (194.0, 68.5)
- removed the ? at (194.0, 73.0)
- removed the ? at (194.0, 71.5)
- removed the ? at (194.0, 70.0)
- removed the ? at (194.0, 58.0)
- removed the ? at (194.0, 59.5)
- removed the ? at (194.0, 61.0)
- removed the ? at (194.0, 56.5)
- removed the ? at (197.0, 50.5)
- removed the ? at (195.5, 50.5)
- removed the ? at (194.0, 50.5)
- removed the ? at (194.0, 55.0)
- removed the ? at (194.0, 53.5)
- removed the ? at (194.0, 52.0)
- removed the ? at (201.5, 50.5)
- removed the ? at (194.0, 26.5)
- removed the ? at (200.0, 50.5)
- removed the ? at (198.5, 50.5)
- removed the ? at (203.0, 50.5)
- removed the ? at (204.5, 50.5)
- removed the ? at (206.0, 50.5)
- removed the ? at (224.0, 50.5)
- removed the ? at (222.5, 50.5)
- removed the ? at (221.0, 50.5)
- removed the ? at (216.5, 50.5)
- removed the ? at (218.0, 50.5)
- removed the ? at (194.0, 28.0)
- removed the ? at (219.5, 50.5)
- removed the ? at (210.5, 50.5)
- removed the ? at (209.0, 50.5)
- removed the ? at (207.5, 50.5)
- removed the ? at (212.0, 50.5)
- removed the ? at (213.5, 50.5)
- removed the ? at (215.0, 50.5)
- removed the ? at (194.0, 29.5)
- removed the ? at (194.0, 31.0)
- removed the ? at (194.0, 35.5)
- removed the ? at (194.0, 34.0)
- removed D14, D15, D16: CONN_01X03, Pin_Headers:Pin_Header_Straight_1x03_Pitch2.54mm
- removed PWM1: CONN_01X06, Pin_Headers:Pin_Header_Straight_1x06_Pitch2.54mm
- added (IN)D14: CONN_01X03, Pin_Headers:Pin_Header_Straight_1x03_Pitch2.54mm, F.Cu at (163.1, 57.9)
- added 0.1uF3: 0.1uF, Capacitors_THT:C_Rect_L4.0mm_W2.5mm_P2.50mm, F.Cu at (164.0, 27.0)
- added 1k6: 1k, Resistors_THT:R_Axial_DIN0204_L3.6mm_D1.6mm_P2.54mm_Vertical, F.Cu at (155.0, 41.8)
- added 2.2k6: 2.2k, Resistors_THT:R_Axial_DIN0204_L3.6mm_D1.6mm_P2.54mm_Vertical, F.Cu at (156.0, 62.8)
- added 3.3k2: 3.3k, Resistors_THT:R_Axial_DIN0204_L3.6mm_D1.6mm_P2.54mm_Vertical, F.Cu at (156.0, 60.4)
- added 47uF10V2: 47uF 10V, Capacitors_THT:CP_Radial_D8.0mm_P2.50mm, F.Cu at (147.0, 31.0)
- added D11: CONN_01X03, Pin_Headers:Pin_Header_Straight_1x03_Pitch2.54mm, F.Cu at (171.0, 68.0)
- added D3: CONN_01X03, Pin_Headers:Pin_Header_Straight_1x03_Pitch2.54mm, F.Cu at (139.0, 68.0)
- added D5: CONN_01X03, Pin_Headers:Pin_Header_Straight_1x03_Pitch2.54mm, F.Cu at (147.0, 68.0)
- added D6: CONN_01X03, Pin_Headers:Pin_Header_Straight_1x03_Pitch2.54mm, F.Cu at (151.0, 68.0)
- added Rx_Tx_Gnd5V1: CONN_01X04, Pin_Headers:Pin_Header_Straight_1x04_Pitch2.54mm, F.Cu at (145.0, 63.0)
- added U1: LM7805CT, Power_Integrations:TO-220, F.Cu at (157.0, 28.0)
- 0.1uF1, 0.1uF2, 0.1uF5, 0.1uF6, 22pF1, 22pF2: footprint Capacitors_ThroughHole:C_Rect_L4.0mm_W2.5mm_P2.50mm -> Capacitors_THT:C_Rect_L4.0mm_W2.5mm_P2.50mm
- 10k1, 10k2, 10k3, 10k5, 1k1, 1k2, 1k3, 1k4, 1k5, 1k7, 1k8, 2.2k1, 2.2k2, 2.2k3, 2.2k4, 2.2k5, 3.3k1: footprint Resistors_ThroughHole:R_Axial_DIN0204_L3.6mm_D1.6mm_P2.54mm_Vertical -> Resistors_THT:R_Axial_DIN0204_L3.6mm_D1.6mm_P2.54mm_Vertical
- 47uF10V1: footprint Capacitors_ThroughHole:CP_Radial_D8.0mm_P2.50mm -> Capacitors_THT:CP_Radial_D8.0mm_P2.50mm
- Rx_Tx_Gnd5V1: renamed from RX TX GND 5V
- moved 10k1 22.6 mm to (172.0, 31.0)
- moved 6V-IN1 22.4 mm to (169.0, 28.0), turned to 0 degrees
- moved 10k3 22.2 mm to (172.0, 28.0)
- moved GrI2C-S1 22.2 mm to (128.0, 60.3), turned to 0 degrees
- moved 1k8 19.5 mm to (152.4, 59.8)
- moved D12 16.0 mm to (175.0, 68.0)
- moved D13 16.0 mm to (179.0, 68.0)
- moved 2.2k3 15.9 mm to (138.0, 61.0), turned to 270 degrees
- moved 2.2k2 15.0 mm to (135.0, 61.0), turned to 270 degrees
- moved 1k3 12.8 mm to (159.6, 41.8)
- moved D10 12.0 mm to (167.0, 68.0)
- moved D7 12.0 mm to (155.0, 68.0)
- moved D8 12.0 mm to (159.0, 68.0)
- moved D9 12.0 mm to (163.0, 68.0)
- moved 1k4 7.02 mm to (188.0, 63.5), turned to 0 degrees
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- renumbered BT-5V1 to 5VGnd_Rx_Tx1, U2 to HC05-06BT1, ISP1 to ISP_D11_D12_D13Rst_5V_Gnd1, UART1 to Rst_Tx_Rx_5V_-_GND1
Connections:
- net Net-(10k3-Pad1) renamed +6V
- 1k3 pad 1: /RXD -> Net-(1k3-Pad1)
- 1k3 pad 2: Net-(1k3-Pad2) -> /RXD
- 1k8 pad 1: Net-(1k8-Pad1) -> /D15/A1
- 1k8 pad 2: /TXD -> Net-(1k8-Pad2)
- 5VGnd_Rx_Tx1 pad 1: Net-(1k8-Pad1) -> Net-(2.2k1-Pad2)
- 5VGnd_Rx_Tx1 pad 2: Net-(1k3-Pad2) -> Net-(1k3-Pad1)
- P1 pad 5: (no net) -> Net-(P1-Pad5)
- RN42XV1 pad 2: Net-(1k3-Pad2) -> Net-(1k3-Pad1)
- Rst_Tx_Rx_5V_-_GND1 pad 2: /TXD -> Net-(1k6-Pad1)
- Rst_Tx_Rx_5V_-_GND1 pad 3: /RXD -> Net-(1k3-Pad1)
Routing:
- net Net-(1k3-Pad1): track 0.00 -> 50.6 mm
- net Net-(1k8-Pad1): track 38.1 -> 0.00 mm
- net Net-(1k3-Pad2): track 33.1 -> 0.00 mm
- net Net-(2.2k3-Pad2): track 15.5 -> 38.8 mm
- net Net-(2.2k2-Pad2): track 18.3 -> 38.4 mm
- net /RXD: track 23.7 -> 6.24 mm
- net /D5(P): track 9.81 -> 21.2 mm
- net Net-(2.2k1-Pad2): track 17.5 -> 28.2 mm
- net +6V: track 3.20 -> 13.3 mm
- net /D3(P): track 21.4 -> 31.3 mm
- net /D14/A0: track 21.8 -> 12.0 mm
- net /D8: track 23.8 -> 14.0 mm
- net Net-(2.2k6-Pad1): track 0.00 -> 9.73 mm
- net /D7: track 25.9 -> 16.2 mm
- net GND: track 323.1 -> 332.5 mm
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- added copper zone on B.Cu, net GND
- added copper zone on F.Cu, net GND
Other:
- outline, holes or cut-outs redrawn
- board text added: ">5V"
- board text added: ">Gnd"
- board text added: "GND"
- board text added: "Only328PB"
- board text added: "↓NotPB"
