File: KICAD/droidrone.sch (KiCad schematic (older format))
At the start: 68 parts, among them IC1 ATMEGA328PB, P1 USB_A, U1 TA4805S, U2 ITEAD_HC-05, U4 LP2950L-3.3V, Y1 Crystal

Commit message: chg sch
Parts:
- removed 0.1uF4: 0.1uF, Capacitors_ThroughHole:C_Rect_L4.0mm_W2.5mm_P2.50mm, symbol C
- removed 100uF10V1: 100uF 10V, Capacitors_ThroughHole:CP_Radial_D8.0mm_P2.50mm, symbol CP1
- removed 10k4: 10k, Resistors_ThroughHole:R_Axial_DIN0204_L3.6mm_D1.6mm_P2.54mm_Vertical, symbol R
- removed 1k6: 1k, Resistors_ThroughHole:R_Axial_DIN0204_L3.6mm_D1.6mm_P2.54mm_Vertical, symbol R
- removed D17: CONN_01X03, Pin_Headers:Pin_Header_Straight_1x03_Pitch2.54mm, symbol CONN_01X03
- removed HC05S1: LED, LEDs:LED_D5.0mm, symbol LED
- removed No-BEC1: JUMPER, Pin_Headers:Pin_Header_Straight_1x02_Pitch2.54mm, symbol JUMPER
- removed U1: TA4805S, TO_SOT_Packages_THT:TO-220_Neutral123_Vertical_LargePads, symbol 7805-RESCUE-droidrone
Connections:
- net +5VA is gone; now on net +5V: D10.2 (P2), D12.2 (P2), D13.2 (P2), D2.2 (P2), D4.2 (P2), D7.2 (P2), D8.2 (P2), D9.2 (P2)
- net +5V: now also 2.2k3.1; no longer 2.2k3.2
- net at GrI2C-S1.3 (P3), IC1.3 (PE0(SDA1/ICP4/ACO/PTCXY)): now also 2.2k3.2; no longer 2.2k3.1
- net +6V: no longer names the net of 10k3.1, 6V-IN1.1 (P1)
Other:
- moved on the sheet: 10k1, 10k3, 2.2k2, 2.2k3, 6V-IN1, D2, D4, D7, GrI2C-S1

Commit message: 配線開始
Parts:
- 6V-IN1: footprint lib:TB-2pin -> Pin_Headers:Pin_Header_Straight_1x02_Pitch2.54mm
Connections:
- net GND: now also 22pF2.2; no longer 22pF2.1
- net at IC1.8 ((XTAL2/TOSC2)PB7), Y1.1: now also 22pF2.1; no longer 22pF2.2

Commit message: 配線終了2
Parts:
- removed PWM1: CONN_01X06, Pin_Headers:Pin_Header_Straight_1x06_Pitch2.54mm, symbol CONN_01X06
- added 0.1uF3: 0.1uF, Capacitors_THT:C_Rect_L4.0mm_W2.5mm_P2.50mm, symbol C
- added 1k6: 1k, Resistors_THT:R_Axial_DIN0204_L3.6mm_D1.6mm_P2.54mm_Vertical, symbol R
- added 2.2k6: 2.2k, Resistors_THT:R_Axial_DIN0204_L3.6mm_D1.6mm_P2.54mm_Vertical, symbol R
- added 3.3k2: 3.3k, Resistors_THT:R_Axial_DIN0204_L3.6mm_D1.6mm_P2.54mm_Vertical, symbol R
- added 47uF10V2: 47uF 10V, Capacitors_THT:CP_Radial_D8.0mm_P2.50mm, symbol CP1
- added D11, D2: CONN_01X03, Pin_Headers:Pin_Header_Straight_1x03_Pitch2.54mm, symbol CONN_01X03
- added Rx_Tx_Gnd5V1: CONN_01X04, Pin_Headers:Pin_Header_Straight_1x04_Pitch2.54mm, symbol CONN_01X04
- added U1: LM7805CT, Power_Integrations:TO-220, symbol LM7805CT
- 0.1uF1, 0.1uF2, 0.1uF5, 0.1uF6, 22pF1, 22pF2: footprint Capacitors_ThroughHole:C_Rect_L4.0mm_W2.5mm_P2.50mm -> Capacitors_THT:C_Rect_L4.0mm_W2.5mm_P2.50mm
- 10k1, 10k2, 10k3, 10k5, 1k1, 1k2, 1k3, 1k4, 1k5, 1k7, 1k8, 2.2k1, 2.2k2, 2.2k3, 2.2k4, 2.2k5, 3.3k1: footprint Resistors_ThroughHole:R_Axial_DIN0204_L3.6mm_D1.6mm_P2.54mm_Vertical -> Resistors_THT:R_Axial_DIN0204_L3.6mm_D1.6mm_P2.54mm_Vertical
- 47uF10V1: footprint Capacitors_ThroughHole:CP_Radial_D8.0mm_P2.50mm -> Capacitors_THT:CP_Radial_D8.0mm_P2.50mm
- Conn1, L-D13, Pow1, State1, WakeUp1: symbol LED -> LED-RESCUE-droidrone
- P1: symbol USB_A -> USB_A-RESCUE-droidrone
- Y1: footprint Crystals:Crystal_HC49-U-3pin_Vertical -> lib:Crystal_HC49-U-3pin_Vertical
- renumbered D14 to (IN)D14, BT-5V1 to 5VGnd_Rx_Tx1, D15 to D3, D16 to D4, D2 to D5, D4 to D6, U2 to HC05-06BT1, ISP1 to ISP_D11_D12_D13Rst_5V_Gnd1, UART1 to Rst_Tx_Rx_5V_-_GND1, SPP5V1 to Rx_Tx_Gnd5V1
Connections:
- net +5V: now also 47uF10V2.1, D11.2 (P2), D2.2 (P2), Rx_Tx_Gnd5V1.4 (P4), U1.3 (OUT)
- net D11(P): now also D11.1 (P1)
- net D15/A1: now also 1k8.1; no longer D3.1 (P1)
- net D16/A2: now also 2.2k6.2, 3.3k2.2; no longer D4.1 (P1)
- net D2: now also D2.1 (P1); no longer D5.1 (P1)
- net D3(P): now also D3.1 (P1)
- net D4: now also D4.1 (P1); no longer D6.1 (P1)
- net D5(P): now also D5.1 (P1)
- net D6(P): now also D6.1 (P1)
- net GND: now also 0.1uF3.2, 3.3k2.1, 47uF10V2.2, D11.3 (P3), D2.3 (P3), Rx_Tx_Gnd5V1.3 (P3), U1.2 (GND)
- net RXD: now also 1k3.2; no longer 1k3.1, Rst_Tx_Rx_5V_-_GND1.3 (P3)
- net TXD: now also 1k6.2; no longer 1k8.2, Rst_Tx_Rx_5V_-_GND1.2 (P2)
- net +6V: now reaches 10k3.1, 6V-IN1.1 (P1)
- net +6V: now also 0.1uF3.1, U1.1 (IN)
- net at 5VGnd_Rx_Tx1.2 (P2), RN42XV1.2 (TXD): now also 1k3.1, Rst_Tx_Rx_5V_-_GND1.3 (P3); no longer 1k3.2
- net at 2.2k1.2, 3.3k1.2, RN42XV1.3 (RXD): now also 5VGnd_Rx_Tx1.1 (P1)
- new net: 1k6.1, Rst_Tx_Rx_5V_-_GND1.2 (P2)
- new net: 2.2k6.1, Rx_Tx_Gnd5V1.2 (P2)
- new net: 1k8.2, Rx_Tx_Gnd5V1.1 (P1)
Other:
- note added: "Not328PB,NoUseGrI2C,No2.2k3->GND"
- moved on the sheet: (IN)D14, 1k3, 2.2k1, 3.3k1, 5VGnd_Rx_Tx1, D10, D12, D13, D3, D4, D5, D6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
